Commit message: Can start sim with Iris using run_sim bash script

File: catkin_ws/src/sim_mbr/models/aerial_manipulator.urdf.xacro (robot description, xacro)
@@ -1,5 +1,5 @@
-<?xml version="1.0">
+<?xml version="1.0"?>
 <!-- This file combines all the parts to create the full aerial manipulator robot description -->
-<robot xmlns:xacro="http://www.ros.org/wiki/xacro" name="element">
+<robot xmlns:xacro="http://www.ros.org/wiki/xacro" name="mbr_vehicle">
   <xacro:include filename="parameters.xacro" />
   <xacro:include filename="utils.xacro" />
@@ -22,3 +22,13 @@
     </inertial>
   </link>
+  <!-- Revolute joint with AoR parallel to platform NED y-axis, between platform and manipulator-->
+  <joint name="tilt_servo" type="revolute">
+  # Fill this in
+  </joint>
+  <!-- Link ROS to Gazebo -->
+  <gazebo>
+    <plugin name="gazebo_ros_control" filename="libgazebo_ros_control.so">
+      <robotNamespace>/</robotNamespace>
+    </plugin>
+  </gazebo>
 </robot>

File: catkin_ws/src/sim_mbr/models/aerial_platform.xacro (robot description, xacro)
@@ -1,3 +1,3 @@
-<?xml version="1.0">
+<?xml version="1.0"?>
 <!-- This file specifies the links and joints that make up the aerial platform. It uses helper macros from utils.xacro and takes parameters from parameters.xacro -->
   <xacro:include filename="parameters.xacro" />

File: catkin_ws/src/sim_mbr/models/delta_manipulator.xacro (robot description, xacro)
@@ -1,15 +1,122 @@
-<?xml version="1.0">
+<?xml version="1.0"?>
 <!-- This file specifies the structure of the delta manipulator. It uses helper macros from the utils xacro and takes parameters from the parameters xacro file. -->
+<robot xmlns:xacro="http://www.ros.org/wiki/xacro" name="delta_manipulator">
   <xacro:include filename="parameters.xacro" />
   <xacro:include filename="utils.xacro" />
-  <!-- Create 3x bicep -->
-  <xacro:cylinder name="bicep_1" radius="${radius_element}" length="${length_bicep}">
-  <xacro:cylinder name="bicep_2" radius="${radius_element}" length="${length_bicep}">
-  <xacro:cylinder name="bicep_3" radius="${radius_element}" length="${length_bicep}">
-  <!-- Create 3x forearm -->
-  <xacro:cylinder name="forearm_1" radius="${radius_element}" length="${length_forearm}">
-  <xacro:cylinder name="forearm_2" radius="${radius_element}" length="${length_forearm}">
-  <xacro:cylinder name="forearm_3" radius="${radius_element}" length="${length_forearm}">
-  <!-- Create base and ee -->
-  <xacro:cylinder name="base" radius="${radius_base}" length="${thickness_base}">
-  <xacro:cylinder name="end_effector" radius="${radius_ee}" length="${thickness_ee}">
+  <!-- Links -->
+  <!-- Bicep links -->
+  <xacro:cylinder name="bicep_1" radius="${radius_element}" length="${length_bicep}" mass="${mass}" />
+  <xacro:cylinder name="bicep_2" radius="${radius_element}" length="${length_bicep}" mass="${mass}" />
+  <xacro:cylinder name="bicep_3" radius="${radius_element}" length="${length_bicep}" mass="${mass}" />
+  <!-- Forearm links -->
+  <xacro:cylinder name="forearm_1" radius="${radius_element}" length="${length_forearm}" mass="${mass}" />
+  <xacro:cylinder name="forearm_2" radius="${radius_element}" length="${length_forearm}" mass="${mass}" />
+  <xacro:cylinder name="forearm_3" radius="${radius_element}" length="${length_forearm}" mass="${mass}" />
+  <!-- Base and ee links -->
+  <xacro:cylinder name="base" radius="${radius_base}" length="${thickness_base}" mass="${mass}" />
+  <xacro:cylinder name="end_effector" radius="${radius_ee}" length="${thickness_ee}" mass="${mass}" />
+  <!-- Elbow joint links -->
+  <xacro:univ_joint name="elbow_1" />
+  <xacro:univ_joint name="elbow_2" />
+  <xacro:univ_joint name="elbow_3" />
+  <!-- Wrist joint links -->
+  <xacro:univ_joint name="wrist_1" />
+  <xacro:univ_joint name="wrist_2" />
+  <xacro:univ_joint name="wrist_3" />
+  <!-- Joints -->
+  <!-- Revolute joints between base and biceps -->
+  <joint name="base_to_bicep_1" type="revolute">
+    <parent link="base" />
+    <child  link="bicep_1" />
+    <axis />
+    <origin xyz="" rpy ="" />
+  </joint>
+  <joint name="base_to_bicep_2" type="revolute">
+    <parent link="base" />
+    <child  link="bicep_2" />
+    <axis />
+    <origin xyz="" rpy ="" />
+  </joint>
+  <joint name="base_to_bicep_3" type="revolute">
+    <parent link="base" />
+    <child  link="bicep_3" />
+    <axis />
+    <origin xyz="" rpy ="" />
+  </joint>
+  <!-- Continuous joints between biceps and universal elbow joint link -->
+  <joint name="bicep_to_elbow_1" type="continuous">
+    <parent link="bicep_1" />
+    <child  link="elbow_1" />
+    <axis />
+    <origin xyz="" rpy="" />
+  </joint>
+  <joint name="bicep_to_elbow_2" type="continuous">
+    <parent link="bicep_2" />
+    <child  link="elbow_2" />
+    <axis />
+    <origin xyz="" rpy="" />
+  </joint>
+  <joint name="bicep_to_elbow_3" type="continuous">
+    <parent link="bicep_3" />
+    <child  link="elbow_3" />
+    <axis />
+    <origin xyz="" rpy="" />
+  </joint>
+  <!-- Continuous joints between universal elbow joint links and forearm -->
+    <joint name="elbow_to_forearm_1" type="continuous">
+    <parent link="elbow_1" />
+    <child  link="forearm_1" />
+    <axis />
+    <origin xyz="" rpy="" />
+  </joint>
+  <joint name="elbow_to_forearm_2" type="continuous">
+    <parent link="elbow_2" />
+    <child  link="forearm_2" />
+    <axis />
+    <origin xyz="" rpy="" />
+  </joint>
+  <joint name="elbow_to_forearm_3" type="continuous">
+    <parent link="elbow_3" />
+    <child  link="forearm_3" />
+    <axis />
+    <origin xyz="" rpy="" />
+  </joint>
+  <!-- Continuous joints between forearms and universal wrist joint link -->
+  <joint name="forearm_to_wrist_1" type="continuous">
+    <parent link="forearm_1" />
+    <child  link="wrist_1" />
+    <axis />
+    <origin xyz="" rpy="" />
+  </joint>
+  <joint name="forearm_to_wrist_2" type="continuous">
+    <parent link="forearm_2" />
+    <child  link="wrist_2" />
+    <axis />
+    <origin xyz="" rpy="" />
+  </joint>
+  <joint name="forearm_to_wrist_3" type="continuous">
+    <parent link="forearm_3" />
+    <child  link="wrist_3" />
+    <axis />
+    <origin xyz="" rpy="" />
+  </joint>
+  <!-- Continuous joints between universal wrist joint link and ee -->
+  <joint name="wrist_to_ee_1" type="continuous">
+    <parent link="wrist_1" />
+    <child  link="end_effector" />
+    <axis />
+    <origin xyz="" rpy="" />
+  </joint>
+  <joint name="wrist_to_ee_2" type="continuous">
+    <parent link="wrist_2" />
+    <child  link="end_effector" />
+    <axis />
+    <origin xyz="" rpy="" />
+  </joint>
+  <joint name="wrist_to_ee_3" type="continuous">
+    <parent link="wrist_3" />
+    <child  link="end_effector" />
+    <axis />
+    <origin xyz="" rpy="" />
+  </joint>
+</robot>

File: catkin_ws/src/sim_mbr/models/parameters.xacro (robot description, xacro)
@@ -1,3 +1,3 @@
-<?xml version="1.0">
+<?xml version="1.0"?>
 <!-- This file specifies all the configurable parameters that dictate the design of the aerial manipulator. -->
 <robot xmlns:xacro="http://www.ros.org/wiki/xacro">
@@ -8,7 +8,9 @@
   <xacro:property name="radius_base"    value="0.1"   />
   <xacro:property name="radius_ee"      value="0.05"  />
-  <xacro:property name="length_uj"      value="radius_element"  />
-  <xacro:property name="thickness_base" value="0.1*radius_base" />
-  <xacro:property name="thickness_ee"   value="0.1*radius_ee" />
+  <xacro:property name="length_uj"      value="${radius_element}"  />
+  <xacro:property name="mass_uj"        value="0.01" />
+  <xacro:property name="thickness_base" value="${0.1 * radius_base}" />
+  <xacro:property name="thickness_ee"   value="${0.1 * radius_ee}" />
+  <xacro:property name="mass"           value="1.0" /> #Just give every link a mass of 1 for now, add specific masses to increase fidelity
   # Maybe some actuator joint limits?
 </robot>

File: catkin_ws/src/sim_mbr/models/utils.xacro (robot description, xacro)
@@ -1,57 +1,57 @@
-<?xml version="1.0">
+<?xml version="1.0"?>
 <!-- This file specifies the helper macros used in the aerial platform and delta manipulator xacro files -->
 <robot xmlns:xacro="http://www.ros.org/wiki/xacro">
   <!-- Create cylinder element macro -->
-  <xacro:macro name="cylinder" params="name radius length">
+  <xacro:macro name="cylinder" params="name radius length mass element_color:=White">
     <link name="${name}">
       <visual>
         <geometry>
-          <cylinder radius="${radius}" length="${length}">
+          <cylinder radius="${radius}" length="${length}" />
         </geometry>
-        <origin xyz="" rpy=""/> # Fill in
+        <origin xyz="0 0 0" rpy="0 0 0" /> # Fill in
       </visual>
       <collision>
         <geometry>
-          <cylinder radius="${radius}" length="${length}">
+          <cylinder radius="${radius}" length="${length}" />
         </geometry>
-        <origin xyz="" rpy=""/> # Fill in
+        <origin xyz="0 0 0" rpy=" 0 0 0" /> # Fill in
       </collision>
-      <xacro:cylinder_inertial  m="${mass}" # Write cylinder inertial macro in utils
-                                radius="${radius}"
-                                length="${length}"/>
+      <xacro:cylinder_inertial  m="${mass}" x="0" y="0" z="0"
+                                r="${radius}"
+                                l="${length}" />
     </link>
     <!-- Gazebo simulation settings -->
-    <gazebo reference="${name}_${arm_number}">
+    <gazebo reference="${name}">
         <selfCollide>true</selfCollide>
         <static>false</static>
         <turnGravityOff>true</turnGravityOff>
-        <material>Gazebo/${element_colour}</material>
+        <material>Gazebo/${element_color}</material>
     </gazebo>
   </xacro:macro>
   <!-- Universal joint element macro - URDF has no universal joints so we use two revolute/continuous joints around a small, collisionless and inertia-less cube -->
-  <xacro:macro name="univ_joint" params="name arm_number">
-    <link name="${name}_${arm_number}">
+  <xacro:macro name="univ_joint" params="name element_color:=Blue">
+    <link name="${name}">
       <visual>
         <geometry>
-          <box size="${lenght_uj} ${lenght_uj} ${lenght_uj}">
+          <box size="${length_uj} ${length_uj} ${length_uj}" />
         </geometry>
-        <origin xyz="" rpy="" /> # Fill in
+        <origin xyz="0 0 0" rpy="0 0 0" /> # Fill in
       </visual>
       <collision>
-        <origin xyz="" rpy="" /> # Fill in
+        <origin xyz="0 0 0" rpy="0 0 0" /> # Fill in
       </collision>
       <inertial>
-        <mass />
+        <mass value="${mass_uj}" />
       </inertial>
     </link>
-    <gazebo reference="${name}_${arm_number}">
+    <gazebo reference="${name}">
       <selfCollide>true</selfCollide>
       <static>false</static>
       <turnGravityOff>true</turnGravityOff>
-      <material>Gazebo/${element_colour}</material>
+      <material>Gazebo/${element_color}</material>
     </gazebo>
   </xacro:macro>
   <!-- Macro for calculating the <inertial> tag for a box geometry -->
-  <xacro:macro name="box_inertial"params="m x y z dx dy dz">
+  <xacro:macro name="box_inertial" params="m x y z dx dy dz">
     <inertial>
       <mass  value="${m}"/>
@@ -67,7 +67,8 @@
       <mass value="${m}" />
       <origin xyz="${x} ${y} ${z}" rpy="0 0 0" />
-      <inertia  ixx="" ixy="0.0" ixz="0.0" # Fill in inertia calculations
-                iyy="" iyz="0.0"
-                izz="" />
+      <inertia  ixx="${m/12 * (3*r*r + l*l)}" ixy="0.0" ixz="0.0"
+                iyy="${m/2 * (r*r)}" iyz="0.0"
+                izz="${ m/12 * (3*r*r + l*l) }" />
     </inertial>
   </xacro:macro>
+</robot>
